Commit message: 实机开发基线：清理仿真并接入 FAST-LIO 与 JD03 双里程计
移除 Gazebo、演示地图、测试视频回退和模拟巡检执行，保留实机业务接口。
移植速腾/维特 FAST-LIO2 建图与 PCD 全局定位，补齐三维转扫描、Nav2 和地图导出。
接入 JD03 Twist/Ecu 适配、控制仲裁和独立轮速里程计，支持 LIO/轮速/轮速+IMU 选择。
新增统一使用手册、实机移植和底盘里程计说明，保留新车待标定配置及相机能力检查记录。

验证：12 个相关包构建安装通过；16 项离线回归检查通过；原生地图与轮速 ROS 消息收发验证通过。
尚未进行实机运动验证，新车外参、车体几何、底盘反馈比例和运行依赖仍需确认。

File: ros2_ws/src/chassis_description/urdf/chassis.urdf (robot description, URDF)
Before this commit: robot chassis, 9 links, 8 joints
Links:
- removed link Frame
- added link base_link, mass 1.5731528453802; collision mesh filename=package://chassis_description/meshes/Frame.STL; visual mesh filename=package://chassis_description/meshes/Frame.STL
Joints:
- joint steering_1_joint: parent Frame -> base_link
- joint steering_2_joint: parent Frame -> base_link
- joint steering_3_joint: parent Frame -> base_link
- joint steering_4_joint: parent Frame -> base_link
